File: Keyboard/PCB/DSKY_keyboard/DSKY_keyboard.kicad_pcb (KiCad board)
At the start: 2 copper layers, 168.4 x 69.6 mm, 56 parts, among them J1 Conn_01x04_Male, J2 MOUNTINGHOLE3.0, J3 MOUNTINGHOLE3.0, J4 MOUNTINGHOLE3.0, J5 MOUNTINGHOLE3.0, SW1 SW_SPST_LED, SW10 SW_SPST_LED, SW11 SW_SPST_LED, SW12 SW_SPST_LED, SW13 SW_SPST_LED, SW14 SW_SPST_LED, SW15 SW_SPST_LED, SW16 SW_SPST_LED, SW17 SW_SPST_LED, SW18 SW_SPST_LED, SW19 SW_SPST_LED, SW2 SW_SPST_LED, SW20 SWITCH_TACT_SMT4.6X2.8, SW3 SW_SPST_LED, SW4 SW_SPST_LED, SW5 SW_SPST_LED, SW6 SW_SPST_LED, SW7 SW_SPST_LED, SW8 SW_SPST_LED, SW9 SW_SPST_LED, U1 STM32F042K6T6, U2 AQY232SZ, U3 AP2112K-3.3

Commit message: Updated PCB
Parts:
- moved J3 0.13 mm to (182.1, 69.0)
Routing:
- net Net-(SW7-PadLED+): track 0.00 -> 194.9 mm, vias 0 -> 3
- net GND: track 350.4 -> 308.8 mm

Commit message: PCB updates
Parts:
- removed J3, J4, J5: MOUNTINGHOLE3.0, MountingHole:MountingHole_3.2mm_M3_Pad
- removed REF1 (x2): OSHW-Logo2_9.8x8mm_SilkScreen, Symbol:OSHW-Logo2_9.8x8mm_SilkScreen
- added D22: D_Schottky_30V, Trinket M0 rev D:SOD-123FL, B.Cu at (108.0, 82.1)
- added LA: LOGO, anca:anca, F.Cu at (181.9, 79.9)
- added REF**: OSHW-Logo2_9.8x8mm_SilkScreen, Symbol:OSHW-Logo2_9.8x8mm_SilkScreen, B.Cu at (108.1, 100.5)
- added REF**: OSHW-Logo2_9.8x8mm_SilkScreen, Symbol:OSHW-Logo2_9.8x8mm_SilkScreen, F.Cu at (141.0, 104.8)
- J2: value MOUNTINGHOLE3.0 -> 614105150721; footprint MountingHole:MountingHole_3.2mm_M3_Pad -> Footprints:614105150721; moved to B.Cu
- moved J2 41.2 mm to (132.7, 102.1), turned to 180 degrees
Connections:
- J2 pad 1: (no net) -> VBAT
- SW10 pad LED+: Net-(SW10-PadLED+) -> Net-(SW1-PadLED+)
- SW10 pad LED-: Net-(SW10-PadLED-) -> GND
- SW11 pad LED+: Net-(SW11-PadLED+) -> Net-(SW1-PadLED+)
- SW11 pad LED-: Net-(SW10-PadLED+) -> GND
- SW12 pad LED+: Net-(SW12-PadLED+) -> Net-(SW1-PadLED+)
- SW12 pad LED-: Net-(SW11-PadLED+) -> GND
- SW13 pad LED+: Net-(SW13-PadLED+) -> Net-(SW1-PadLED+)
- SW13 pad LED-: Net-(SW12-PadLED+) -> GND
- SW14 pad LED+: Net-(SW14-PadLED+) -> Net-(SW1-PadLED+)
- SW14 pad LED-: Net-(SW13-PadLED+) -> GND
- SW15 pad LED+: Net-(SW15-PadLED+) -> Net-(SW1-PadLED+)
- SW15 pad LED-: Net-(SW14-PadLED+) -> GND
- SW16 pad LED+: Net-(SW16-PadLED+) -> Net-(SW1-PadLED+)
- SW16 pad LED-: Net-(SW15-PadLED+) -> GND
- SW17 pad LED+: Net-(SW17-PadLED+) -> Net-(SW1-PadLED+)
- SW17 pad LED-: Net-(SW16-PadLED+) -> GND
- SW18 pad LED+: Net-(SW18-PadLED+) -> Net-(SW1-PadLED+)
- SW18 pad LED-: Net-(SW17-PadLED+) -> GND
- SW19 pad LED+: Net-(SW19-PadLED+) -> Net-(SW1-PadLED+)
- SW19 pad LED-: Net-(SW18-PadLED+) -> GND
- SW2 pad LED+: Net-(SW2-PadLED+) -> Net-(SW1-PadLED+)
- SW2 pad LED-: Net-(SW1-PadLED+) -> GND
- SW3 pad LED+: Net-(SW3-PadLED+) -> Net-(SW1-PadLED+)
- SW3 pad LED-: Net-(SW2-PadLED+) -> GND
- SW4 pad LED+: Net-(SW4-PadLED+) -> Net-(SW1-PadLED+)
- SW4 pad LED-: Net-(SW3-PadLED+) -> GND
- SW5 pad LED+: Net-(SW5-PadLED+) -> Net-(SW1-PadLED+)
- SW5 pad LED-: Net-(SW4-PadLED+) -> GND
- SW6 pad LED+: Net-(SW6-PadLED+) -> Net-(SW1-PadLED+)
- SW6 pad LED-: Net-(SW5-PadLED+) -> GND
- SW7 pad LED+: Net-(SW7-PadLED+) -> Net-(SW1-PadLED+)
- SW7 pad LED-: Net-(SW6-PadLED+) -> GND
- SW8 pad LED+: Net-(SW8-PadLED+) -> Net-(SW1-PadLED+)
- SW8 pad LED-: Net-(SW7-PadLED+) -> GND
- SW9 pad LED+: Net-(SW10-PadLED-) -> Net-(SW1-PadLED+)
- SW9 pad LED-: Net-(SW8-PadLED+) -> GND
- U1 pad 14: Net-(U1-Pad14) -> (no net)
- U1 pad 15: Net-(U1-Pad15) -> (no net)
- U1 pad 2: Net-(U1-Pad2) -> (no net)
- U1 pad 21: Net-(U1-Pad21) -> PA11
- U1 pad 22: Net-(U1-Pad22) -> PA12
- U1 pad 25: Net-(U1-Pad25) -> (no net)
- U1 pad 26: Net-(U1-Pad26) -> (no net)
- U1 pad 27: Net-(U1-Pad27) -> (no net)
- U1 pad 28: Net-(U1-Pad28) -> (no net)
- U1 pad 29: Net-(U1-Pad29) -> (no net)
- U1 pad 3: Net-(U1-Pad3) -> (no net)
- U1 pad 30: Net-(U1-Pad30) -> (no net)
- U1 pad 31: Net-(U1-Pad31) -> (no net)
- U2 pad 4: Net-(SW19-PadLED+) -> Net-(SW1-PadLED+)
- U3 pad 4: Net-(U3-Pad4) -> (no net)
Routing:
- net Net-(SW1-PadLED+): track 34.9 -> 624.0 mm, vias 1 -> 5
- net GND: track 308.8 -> 688.5 mm, vias 12 -> 14
- net Net-(SW19-PadLED+): track 195.2 -> 0.00 mm, vias 3 -> 0
- net Net-(SW7-PadLED+): track 194.9 -> 0.00 mm, vias 3 -> 0
- net Net-(SW14-PadLED+): track 133.0 -> 0.00 mm
- net PA12: track 0.00 -> 74.3 mm, vias 0 -> 4
- net PA11: track 0.00 -> 73.3 mm, vias 0 -> 1
- net VBAT: track 0.00 -> 42.7 mm, vias 0 -> 1
- net Net-(SW6-PadLED+): track 37.9 -> 0.00 mm
- net Net-(SW8-PadLED+): track 37.0 -> 0.00 mm
- net Net-(SW13-PadLED+): track 32.1 -> 0.00 mm
- net Net-(SW15-PadLED+): track 29.8 -> 0.00 mm
- net Net-(SW5-PadLED+): track 29.5 -> 0.00 mm
- net Net-(SW12-PadLED+): track 28.7 -> 0.00 mm
- net Net-(SW18-PadLED+): track 28.4 -> 0.00 mm
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
Commit message: Update
Parts:
- removed LA: LOGO, anca:anca
- removed the REF** at (108.1, 100.5)
- removed the REF** at (141.0, 104.8)
- added C4: 1uF, Trinket M0 rev D:0603-NO, B.Cu at (175.1, 105.7)
- added C5: 1uF, Trinket M0 rev D:0603-NO, B.Cu at (189.2, 97.1)
- added C6: 1uF, Trinket M0 rev D:0603-NO, B.Cu at (190.4, 106.4)
- added C7: 0.1uF, Trinket M0 rev D:0603-NO, B.Cu at (190.4, 103.9)
- added R3: 100K, Trinket M0 rev D:0603-NO, B.Cu at (183.6, 79.6)
- added REF**: MountingHole_2.2mm_M2, MountingHole:MountingHole_2.2mm_M2, F.Cu at (108.1, 67.9)
- added REF**: MountingHole_2.2mm_M2, MountingHole:MountingHole_2.2mm_M2, F.Cu at (182.0, 67.9)
- added REF**: MountingHole_2.2mm_M2, MountingHole:MountingHole_2.2mm_M2, F.Cu at (182.0, 116.0)
- added REF**: MountingHole_2.2mm_M2, MountingHole:MountingHole_2.2mm_M2, F.Cu at (108.1, 116.0)
- U1: value STM32F042K6T6 -> STM32L082KZT6
- moved R1 107.7 mm to (199.1, 106.3), turned to 0 degrees
- moved C2 88.9 mm to (180.1, 79.6)
- moved C1 85.2 mm to (173.8, 79.6)
- moved C3 81.0 mm to (174.4, 98.6), turned to 180 degrees
- moved R2 80.5 mm to (163.6, 79.6), turned to 270 degrees
- moved U3 77.3 mm to (177.0, 79.6)
- moved U2 74.2 mm to (157.5, 79.6)
- moved D22 60.1 mm to (168.0, 79.6), turned to 90 degrees
- moved RESET1 11.6 mm to (199.1, 103.3), turned to 0 degrees
- moved D20 10.7 mm to (171.2, 79.6), turned to 90 degrees
- moved D13 3.29 mm to (206.7, 86.9), turned to 180 degrees
- moved D6 3.29 mm to (206.7, 72.5), turned to 180 degrees
- moved D19 3.27 mm to (206.8, 111.6), turned to 180 degrees
- moved D14 2.73 mm to (224.2, 94.2), turned to 180 degrees
- turned D1 to 180 degrees
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- renumbered SW20 to RESET1
Connections:
- SW1 pad LED+: Net-(SW1-PadLED+) -> +3V3
- SW1 pad LED-: GND -> Net-(SW1-PadLED-)
- SW10 pad LED+: Net-(SW1-PadLED+) -> +3V3
- SW10 pad LED-: GND -> Net-(SW1-PadLED-)
- SW11 pad LED+: Net-(SW1-PadLED+) -> +3V3
- SW11 pad LED-: GND -> Net-(SW1-PadLED-)
- SW12 pad LED+: Net-(SW1-PadLED+) -> +3V3
- SW12 pad LED-: GND -> Net-(SW1-PadLED-)
- SW13 pad LED+: Net-(SW1-PadLED+) -> +3V3
- SW13 pad LED-: GND -> Net-(SW1-PadLED-)
- SW14 pad LED+: Net-(SW1-PadLED+) -> +3V3
- SW14 pad LED-: GND -> Net-(SW1-PadLED-)
- SW15 pad LED+: Net-(SW1-PadLED+) -> +3V3
- SW15 pad LED-: GND -> Net-(SW1-PadLED-)
- SW16 pad LED+: Net-(SW1-PadLED+) -> +3V3
- SW16 pad LED-: GND -> Net-(SW1-PadLED-)
- SW17 pad LED+: Net-(SW1-PadLED+) -> +3V3
- SW17 pad LED-: GND -> Net-(SW1-PadLED-)
- SW18 pad LED+: Net-(SW1-PadLED+) -> +3V3
- SW18 pad LED-: GND -> Net-(SW1-PadLED-)
- SW19 pad LED+: Net-(SW1-PadLED+) -> +3V3
- SW19 pad LED-: GND -> Net-(SW1-PadLED-)
- SW2 pad LED+: Net-(SW1-PadLED+) -> +3V3
- SW2 pad LED-: GND -> Net-(SW1-PadLED-)
- SW3 pad LED+: Net-(SW1-PadLED+) -> +3V3
- SW3 pad LED-: GND -> Net-(SW1-PadLED-)
- SW4 pad LED+: Net-(SW1-PadLED+) -> +3V3
- SW4 pad LED-: GND -> Net-(SW1-PadLED-)
- SW5 pad LED+: Net-(SW1-PadLED+) -> +3V3
- SW5 pad LED-: GND -> Net-(SW1-PadLED-)
- SW6 pad LED+: Net-(SW1-PadLED+) -> +3V3
- SW6 pad LED-: GND -> Net-(SW1-PadLED-)
- SW7 pad LED+: Net-(SW1-PadLED+) -> +3V3
- SW7 pad LED-: GND -> Net-(SW1-PadLED-)
- SW8 pad LED+: Net-(SW1-PadLED+) -> +3V3
- SW8 pad LED-: GND -> Net-(SW1-PadLED-)
- SW9 pad LED+: Net-(SW1-PadLED+) -> +3V3
- SW9 pad LED-: GND -> Net-(SW1-PadLED-)
- U1 pad 16: Net-(C3-Pad1) -> GND
- U1 pad 25: (no net) -> Net-(C3-Pad1)
- U1 pad 31: (no net) -> Net-(R3-Pad2)
- U1 pad 32: Net-(C3-Pad1) -> GND
- U2 pad 4: Net-(SW1-PadLED+) -> Net-(SW1-PadLED-)
Routing:
- net Net-(SW1-PadLED+): track 624.0 -> 0.00 mm, vias 5 -> 0
- net Net-(SW1-PadLED-): track 0.00 -> 533.7 mm, vias 0 -> 7
- net +3V3: track 128.6 -> 657.6 mm, vias 3 -> 11
- net GND: track 688.5 -> 287.8 mm, vias 14 -> 15
- net Net-(D21-Pad2): track 232.7 -> 23.1 mm, vias 4 -> 2
- net Net-(C3-Pad1): track 126.6 -> 4.30 mm, vias 6 -> 0
- net Net-(C1-Pad1): track 83.8 -> 12.8 mm, vias 2 -> 0
- net Net-(R2-Pad2): track 114.4 -> 66.0 mm, vias 2 -> 4
- net Net-(R3-Pad2): track 0.00 -> 22.4 mm, vias 0 -> 2
- net PA02: track 108.4 -> 126.2 mm, vias 0 -> 2
- net VBAT: track 42.7 -> 58.1 mm
- net VBUS: track 20.1 -> 33.9 mm, vias 1 -> 3
- net PA08: track 63.3 -> 74.2 mm
- net /~RESET: track 12.5 -> 23.1 mm
- net PA11: track 73.3 -> 63.9 mm
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Other:
- board text added: "DSKY Keyboard (Cherry MX) Rev. B02"
- board text added: "Designed by Vlad Mihailescu in Canada"
- board text removed: "DSKY Keyboard (Cherry MX) V1 Designed by Vlad Mihailescu"
